File: pcb/shortypcb.kicad_sch (KiCad schematic)
At the start: 14 parts, among them SW1 SW_SPST, U1 kb2040, U2 2465

Commit message: uhh update june fourteeth
Parts:
- C1, C2, C3, C4: footprint Capacitor_SMD:C_0201_0603Metric_Pad0.64x0.40mm_HandSolder -> CC0402KRX5R5BB105 (2):CAPC1005X60
- Resistor1: footprint Resistor_SMD:R_0603_1608Metric_Pad0.98x0.95mm_HandSolder -> 5-1res:RC0603N_YAG
- Resistor2, Resistor3: footprint Resistor_SMD:R_0603_1608Metric_Pad0.98x0.95mm_HandSolder -> 1mohmres:RES_TLR_3AW1_2_4_KOA
Changed lines of the file:
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@@
 			)
 		)
-		(property "Footprint" "Capacitor_SMD:C_0201_0603Metric_Pad0.64x0.40mm_HandSolder"
+		(property "Footprint" "CC0402KRX5R5BB105 (2):CAPC1005X60"
 			(at 204.47 67.31 0)
 			(effects
@@
 			)
 		)
-		(property "Footprint" "Resistor_SMD:R_0603_1608Metric_Pad0.98x0.95mm_HandSolder"
+		(property "Footprint" "1mohmres:RES_TLR_3AW1_2_4_KOA"
 			(at 194.31 104.648 90)
 			(effects
@@
 			)
 		)
-		(property "Footprint" "Resistor_SMD:R_0603_1608Metric_Pad0.98x0.95mm_HandSolder"
+		(property "Footprint" "1mohmres:RES_TLR_3AW1_2_4_KOA"
 			(at 184.15 104.648 90)
 			(effects
@@
 			)
 		)
-		(property "Footprint" "Capacitor_SMD:C_0201_0603Metric_Pad0.64x0.40mm_HandSolder"
+		(property "Footprint" "CC0402KRX5R5BB105 (2):CAPC1005X60"
 			(at 142.24 107.95 0)
 			(effects
@@
 			)
 		)
-		(property "Footprint" "Capacitor_SMD:C_0201_0603Metric_Pad0.64x0.40mm_HandSolder"
+		(property "Footprint" "CC0402KRX5R5BB105 (2):CAPC1005X60"
 			(at 85.09 132.08 0)
 			(effects
@@
 			)
 		)
-		(property "Footprint" "Resistor_SMD:R_0603_1608Metric_Pad0.98x0.95mm_HandSolder"
+		(property "Footprint" "5-1res:RC0603N_YAG"
 			(at 95.25 51.308 90)
 			(effects
@@
 			)
 		)
-		(property "Footprint" "Capacitor_SMD:C_0201_0603Metric_Pad0.64x0.40mm_HandSolder"
+		(property "Footprint" "CC0402KRX5R5BB105 (2):CAPC1005X60"
 			(at 162.56 93.98 0)
 			(effects
