File: pcb/shortypcb.kicad_pcb (KiCad board)
At the start: 2 copper layers, 93.2 x 24.4 mm, 19 parts, among them SW1 SW_SPST, U1 kb2040, U2 2465

Commit message: uhh update june fourteeth
Parts:
- C1: footprint Capacitor_SMD:C_0201_0603Metric_Pad0.64x0.40mm_HandSolder -> CC0402KRX5R5BB105 (2):CAPC1005X60; moved to B.Cu
- C2, C3, C4: footprint Capacitor_SMD:C_0201_0603Metric_Pad0.64x0.40mm_HandSolder -> CC0402KRX5R5BB105 (2):CAPC1005X60
- Resistor1: footprint Resistor_SMD:R_0603_1608Metric_Pad0.98x0.95mm_HandSolder -> 5-1res:RC0603N_YAG
- Resistor2, Resistor3: footprint Resistor_SMD:R_0603_1608Metric_Pad0.98x0.95mm_HandSolder -> 1mohmres:RES_TLR_3AW1_2_4_KOA
- moved Resistor3 8.45 mm to (138.0, 64.0)
- moved Resistor2 8.03 mm to (146.8, 63.8)
- moved C1 0.94 mm to (125.5, 58.0)
- renumbered OLED1 to OLED
Routing:
- net D+: track 84.1 -> 98.3 mm
- net Net-(U1-A0/26): track 5.55 -> 10.0 mm
- net GND: track 193.8 -> 197.8 mm
- net +3.3V: track 33.3 -> 36.1 mm
- net Net-(U2-VLIPO): track 28.7 -> 30.4 mm, vias 0 -> 2
- net +5V: track 41.8 -> 43.0 mm
- net D-: track 97.4 -> 98.5 mm
- net D8ASSY: track 33.1 -> 33.8 mm

Commit message: PCB is done?
Routing:
- net D-: track 98.5 -> 89.9 mm
- net D+: track 98.3 -> 89.8 mm
- net GND: track 197.8 -> 192.3 mm
- net +3.3V: track 36.1 -> 37.2 mm
- net Net-(U2-VLIPO): track 30.4 -> 29.9 mm
